Commit message: added controllers and arduino files

File: src/trimode/trimode_description/urdf/trimode.urdf.xacro (robot description, xacro)
@@ -128,5 +128,5 @@
 <link name="kinect_link">
   <visual>
-    <origin xyz="0 0 0"/>
+    <origin xyz="0 0 -0.09"/>
     <geometry>
       <!--box size="0.064 0.121 0.0381" /-->
@@ -144,5 +144,5 @@
 </link>
 <joint name="kinect_joint" type="fixed">
-  <origin xyz="0.2 0 0.08" rpy="0 0 0" />
+  <origin xyz="0.2 0 ${0.08 + 0.09}" rpy="0 0 0" />
   <parent link="chassis_link" />
   <child link="kinect_link" />
@@ -251,4 +251,5 @@
   </link>
   <joint name="imu_joint" type="fixed">
+    <origin xyz="0 0 0" rpy="0 0 0"/>
     <parent link="chassis_link" />
     <child link="imu_link" />
